File: KiCad Projects/Uno_Shield_ThermoPro/Uno_Shield_ThermoPro.kicad_pcb (KiCad board)
At the start: 2 copper layers, 68.6 x 53.3 mm, 24 parts, among them J1 Power, J2 Digital/PWM, J3 Analog, J4 Digital/PWM, J5 CONN_GYRO, J6 Connector Display, J7 CONN_TEMP, SW1 SW_SPST, SW2 SW_SPST, SW3 SW_SPST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

Commit message: ThermoPro Project v1
Parts:
- removed MH1, MH2, MH3, MH4: MountingHole_3.2mm, Arduino_MountingHole:MountingHole_3.2mm
- added G***: LOGO, LOGO, F.Cu at (144.0, 92.5)
- R4: value 100k -> 2 x 100k
- R5: value 100k -> 3 x 100k
- moved D1 22.1 mm to (147.7, 54.5)
- moved R5 13.5 mm to (151.1, 66.0)
- moved J7 13.2 mm to (127.0, 64.0)
- moved R3 12.7 mm to (163.5, 69.5)
- moved R1 4.87 mm to (140.9, 59.5), turned to 0 degrees
- moved R4 4.50 mm to (151.4, 82.5)
- moved RV1 2.98 mm to (132.4, 90.5), turned to -90 degrees
- moved R6 2.84 mm to (127.9, 82.5)
- moved SW1 2.25 mm to (154.7, 60.5)
- moved J6 1.77 mm to (117.5, 75.0)
- moved J5 1.46 mm to (103.6, 66.6)
Connections:
- J2 pad 10: /TEMP_DIGITAL -> /8
- J2 pad 5: /13 -> /TEMP_DIGITAL
- J4 pad 2: /BUTTON_UNIT -> /*6
- J4 pad 4: /BUTTON_LIGHT -> /BUTTON_ON/OFF
- J4 pad 5: /BUTTON_ON/OFF -> /BUTTON_LIGHT
- J4 pad 6: /2 -> /BUTTON_UNIT
Routing:
- net /I2C_SCL: track 0.00 -> 42.4 mm
- net /BUTTON_CAL: track 0.00 -> 41.9 mm
- net /BUTTON_UNIT: track 11.2 -> 50.4 mm
- net +5V: track 141.3 -> 177.2 mm
- net /BUTTON_LIGHT: track 0.00 -> 34.7 mm
- net /I2C_SDA: track 0.00 -> 29.9 mm
- net /BUTTON_ON/OFF: track 0.00 -> 25.3 mm
- net /TEMP_SENSOR: track 0.00 -> 17.4 mm
- net /TEMP_DIGITAL: track 0.00 -> 15.5 mm
- net /LED_LIGHT: track 0.00 -> 12.9 mm
- net Net-(D1-A): track 0.00 -> 5.27 mm
- net /BUTTON_LOCK: track 42.0 -> 43.8 mm
Other:
- board text added: "Calibrate"
- board text added: "Light"
- board text added: "Lock"
- board text added: "On/Off"
- board text added: "ThermoPro Temp. Probe v1 Jackson Hall Feb 3, 2025"
- board text added: "­°C/­°F"
