File: KiCad Projects/Uno_Shield_ThermoPro/Uno_Shield_ThermoPro.kicad_sch (KiCad schematic)
At the start: 20 parts, among them J1 Power, J2 Digital/PWM, J3 Analog, J4 Digital/PWM, J5 CONN_GYRO, J6 Connector Display, J7 CONN_TEMP, SW1 SW_SPST, SW2 SW_SPST, SW3 SW_SPST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

Commit message: ThermoPro Project v1
Connections:
- net 13 is gone; now on net TEMP_DIGITAL: J2.5 (Pin_5)
- net 2 is gone; now on net BUTTON_UNIT: J4.6 (Pin_6)
- net BUTTON_LIGHT: now also J4.5 (Pin_5); no longer J4.4 (Pin_4)
- net BUTTON_ON/OFF: now also J4.4 (Pin_4); no longer J4.5 (Pin_5)
- net BUTTON_UNIT: no longer J4.2 (Pin_2)
- net TEMP_DIGITAL: no longer J2.10 (Pin_10)
- new net *6: J4.2 (Pin_2)
- new net 8: J2.10 (Pin_10)
- no-connect marks 19 -> 20
Other:
- note removed: "*6"
- note removed: "8"
Changed lines of the file:
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@@
+	)
+	(no_connect
+		(at 74.93 74.93)
 	)
 	(no_connect
@@
 	)
 	(no_connect
-		(at 74.8942 74.93)
-	)
-	(no_connect
 		(at 21.59 62.23)
 	)
@@
 	)
 	(no_connect
-		(at 74.93 72.39)
+		(at 74.93 62.23)
 	)
 	(no_connect
@@
 	)
 	(no_connect
-		(at 74.93 36.83)
+		(at 74.93 49.53)
 	)
 	(no_connect
@@
 	(no_connect
 		(at 74.93 41.91)
+	)
+	(no_connect
+		(at 74.93 64.77)
 	)
 	(no_connect
@@
 		)
 	)
-	(text "8"
-		(exclude_from_sim no)
-		(at 74.168 48.514 0)
-		(effects
-			(font
-				(size 1.27 1.27)
-			)
-		)
-	)
 	(text "DS18B20\n(TEMP SENSOR)\n"
 		(exclude_from_sim no)
@@
 		(exclude_from_sim no)
 		(at 155.956 61.722 0)
-		(effects
-			(font
-				(size 1.27 1.27)
-			)
-		)
-	)
-	(text "*6\n"
-		(exclude_from_sim no)
-		(at 72.898 61.468 0)
 		(effects
 			(font
@@
 	)
 	(label "BUTTON_ON{slash}OFF"
-		(at 74.93 69.85 0)
+		(at 74.93 67.31 0)
 		(effects
 			(font
@@
 		)
 	)
-	(label "2"
-		(at 74.93 72.39 180)
+	(label "*6"
+		(at 74.93 62.23 180)
 		(effects
 			(font
@@
 		)
 	)
-	(label "13"
-		(at 74.93 36.83 180)
+	(label "8"
+		(at 74.93 49.53 180)
 		(effects
 			(font
@@
 	)
 	(label "TEMP_DIGITAL"
-		(at 74.93 49.53 0)
+		(at 74.93 36.83 0)
 		(effects
 			(font
@@
 	)
 	(label "*5"
-		(at 74.93 64.77 0)
-		(effects
-			(font
-				(size 1.27 1.27)
-			)
-			(justify left bottom)
+		(at 74.93 64.77 180)
+		(effects
+			(font
+				(size 1.27 1.27)
+			)
+			(justify right bottom)
 		)
 	)
@@
 	)
 	(label "BUTTON_UNIT"
-		(at 74.93 62.23 0)
+		(at 74.93 72.39 0)
 		(effects
 			(font
@@
 	)
 	(label "BUTTON_LIGHT"
-		(at 74.93 67.31 0)
-		(effects
-			(font
+		(at 74.93 69.85 0)
+		(effects
+			(font

Commit message: ThermoPro Commit
Other:
- note added: "*2"
- note added: "12"
- note added: "13"
Changed lines of the file:
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@@
+		)
+	)
+	(text "*2"
+		(exclude_from_sim no)
+		(at 73.152 71.374 0)
+		(effects
+			(font
+				(size 1.27 1.27)
+			)
 		)
 	)
@@
 		)
 	)
+	(text "13\n"
+		(exclude_from_sim no)
+		(at 73.406 35.814 0)
+		(effects
+			(font
+				(size 1.27 1.27)
+			)
+		)
+	)
 	(text "* Indicates a PWM-capable pin"
 		(exclude_from_sim no)
@@
 		(effects
 			(font
+				(size 1.27 1.27)
+			)
+		)
+	)
+	(text "12"
+		(exclude_from_sim no)
+		(at 73.406 38.608 0)
+		(effects
+			(font
