File: KiCad Projects/Uno_Shield_FinalProject/Uno_Shield_FinalProject.kicad_pcb (KiCad board)
At the start: 2 copper layers, 68.6 x 53.3 mm, 21 parts, among them J1 Power, J2 Digital/PWM, J3 Analog, J4 Digital/PWM, J7 MPU6050, J8 OpenLog, U1 BME280, U2 TMP36GT9

Commit message: Final Project Commit
Routing:
- net /MISO: track 22.4 -> 0.00 mm
- net /MOSI: track 22.4 -> 0.00 mm
- net /CS: track 22.4 -> 0.00 mm
Changed lines of the file:
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@@
 		)
 		(embedded_fonts no)
+		(model "${KIPRJMOD}/Components/TMP36GT9/TMP36GT9.step"
+			(offset
+				(xyz 0 -1 10.5)
+			)
+			(scale
+				(xyz 1 1 1)
+			)
+			(rotate
+				(xyz -90 -0 -0)
+			)
+		)
 	)
 	(footprint "Resistor_THT:R_Axial_DIN0207_L6.3mm_D2.5mm_P10.16mm_Horizontal"
@@
 		)
 		(embedded_fonts no)
+		(model "${KIPRJMOD}/Components/OpenLog/DEV-13712.step"
+			(offset
+				(xyz 0 0 2.5)
+			)
+			(scale
+				(xyz 1 1 1)
+			)
+			(rotate
+				(xyz -90 -0 -0)
+			)
+		)
 	)
 	(footprint "Resistor_THT:R_Axial_DIN0207_L6.3mm_D2.5mm_P10.16mm_Horizontal"
@@
 	(footprint "2652:MODULE_2652"
 		(layer "F.Cu")
-		(at 121.46 61.515)
+		(at 121.46 61.5)
 		(property "Reference" "U1"
 			(at -5.715 -10.66 0)
@@
 		)
 		(embedded_fonts no)
+		(model "${KIPRJMOD}/Components/BME280/2652.step"
+			(offset
+				(xyz 0 0 1.5)
+			)
+			(scale
+				(xyz 1 1 1)
+			)
+			(rotate
+				(xyz -90 -0 -0)
+			)
+		)
 	)
 	(footprint "LED_THT:LED_D3.0mm"
@@
 		(embedded_fonts no)
 		(model "${KICAD9_3DMODEL_DIR}/Connector_PinSocket_2.54mm.3dshapes/PinSocket_1x08_P2.54mm_Vertical.wrl"
+			(hide yes)
 			(offset
 				(xyz 0 0 0)
@@
 			)
 			(rotate
-				(xyz 0 0 0)
+				(xyz -0 -0 -0)
+			)
+		)
+		(model "C:/Users/Jackson.Hall/Desktop/ENCE_3210_Jackson_Hall/KiCad Projects/Uno_Shield_ThermoPro/Components/MPU6050/ITG-MPU.STEP"
+			(offset
+				(xyz -4 -29.5 -1.5)
+			)
+			(scale
+				(xyz 1 1 1)
+			)
+			(rotate
+				(xyz -90 -0 -180)
 			)
 		)
@@
 		(stroke
 			(width 0.15)
-			(type default)
+			(type solid)
 		)
 		(fill no)
@@
 	)
 	(segment
-		(start 134.036 61.004)
-		(end 134.036 49.2)
-		(width 0.25)
-		(layer "F.Cu")
-		(net 29)
-	)
-	(segment
-		(start 126.54 68.5)
-		(end 134.036 61.004)
-		(width 0.25)
-		(layer "F.Cu")
-		(net 29)
-	)
-	(segment
 		(start 117.70491 49.2)
 		(end 118.796 49.2)
@@
 	)
 	(segment
-		(start 131.496 61.004)
-		(end 124 68.5)
-		(width 0.25)
-		(layer "F.Cu")
-		(net 31)
-	)
-	(segment
-		(start 131.496 49.2)
-		(end 131.496 61.004)
-		(width 0.25)
-		(layer "F.Cu")
-		(net 31)
-	)
-	(segment
 		(start 121.46 56.696)
 		(end 128.956 49.2)
@@
 	)
 	(segment
-		(start 136.576 61.004)
-		(end 136.576 49.2)
-		(width 0.25)
-		(layer "F.Cu")
-		(net 33)
-	)
-	(segment
-		(start 129.08 68.5)
-		(end 136.576 61.004)
-		(width 0.25)
-		(layer "F.Cu")
-		(net 33)
-	)
-	(segment
 		(start 121.336 51.164)
 		(end 110.5 62)
@@
 		(min_thickness 0.25)
 		(filled_areas_thickness no)
-		(fill yes
+		(fill
 			(thermal_gap 0.5)
 			(thermal_bridge_width 0.5)
@@
 		(polygon
 			(pts
-				(xy 95.5 45.5) (xy 172 44.5) (xy 174 105.5) (xy 95 104.5)
+				(xy 95 42.5) (xy 174.5 42.5) (xy 174 105.5) (xy 95 104.5)
 			)
 		)
@@
 		(members "b7cb95b4-199c-4f65-995c-17973d52b2d5" "bd18f46c-b12c-45eb-bb1a-1a056228884d")
 	)
+	(group ""
+		(members "66249f77-b196-40b1-934d-8ff5363f13b8")
+	)
 	(embedded_fonts no)
